File: Schamtic and PCB Girona heatmeasuement/Schamtic and PCB Girona heatmeasuement.kicad_sch (KiCad schematic)
At the start: 0 parts

Commit message: feat(control): add SMART PWM hold mode with visible handover/fallback progress
- Add control modes AUTO/MANUAL/SMART with persisted mode and manual PWM
- Implement SMART supervisor: PID -> learned constant HOLD PWM -> auto fallback to PID on drift
- Add fractional PWM dithering for non-integer hold/manual PWM targets
- Improve SMART stability logic with noise-tolerant decay counter and tuned thresholds
- Make SMART thresholds thermocouple-accuracy aware (0.25 C based bands)
- Emit telemetry for MODE/STATE/MANPWM/HOLDPWM and ENTPROG/EXTPROG/EABS
- Add explicit serial transition logs for SMART enter/exit hold
- Extend GUI with mode controls, manual PWM controls, and SMART live fields
- Add plot series for HOLD PWM, ENTER %, and EXIT %
- Fix GUI bug where telemetry overwrote editable MODE/MANPWM inputs
Parts:
- added U1: ESP32-S3-WROOM-1, RF_Module:ESP32-S3-WROOM-1, symbol RF_Module:ESP32-S3-WROOM-1
Connections:
- new net: U1.1 (GND), U1.40 (GND), U1.41 (GND)
- new net +3.3V: U1.2 (3V3)
Changed lines of the file:
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@@
 	(generator_version "9.0")
 	(paper "A4")
+	(symbol
+		(lib_id "power:+3.3V")
+		(at 125.73 41.91 0)
+		(unit 1)
+		(exclude_from_sim no)
+		(in_bom yes)
+		(on_board yes)
+		(dnp no)
+		(fields_autoplaced yes)
+		(property "Reference" "#PWR01"
+			(at 125.73 45.72 0)
+			(effects
+				(font
+					(size 1.27 1.27)
+				)
+				(hide yes)
+			)
+		)
+		(property "Value" "+3.3V"
+			(at 125.73 36.83 0)
+			(effects
+				(font
+					(size 1.27 1.27)
+				)
+			)
+		)
+		(property "Footprint" ""
+			(at 125.73 41.91 0)
+			(effects
+				(font
+					(size 1.27 1.27)
+				)
+				(hide yes)
+			)
+		)
+		(property "Datasheet" ""
+			(at 125.73 41.91 0)
+			(effects
+				(font
+					(size 1.27 1.27)
+				)
+				(hide yes)
+			)
+		)
+		(property "Description" "Power symbol creates a global label with name \"+3.3V\""
+			(at 125.73 41.91 0)
+			(effects
+				(font
+					(size 1.27 1.27)
+				)
+				(hide yes)
+			)
+		)
+		(pin "1"
+		)
+		(instances
+			(project ""
+				(path "/903e2e1f-69db-4eea-89f5-cdb0bf721490"
+					(reference "#PWR01")
+					(unit 1)
+				)
+			)
+		)
+	)
+	(symbol
+		(lib_id "RF_Module:ESP32-S3-WROOM-1")
+		(at 125.73 69.85 0)
+		(unit 1)
+		(exclude_from_sim no)
+		(in_bom yes)
+		(on_board yes)
+		(dnp no)
+		(fields_autoplaced yes)
+		(property "Reference" "U1"
+			(at 127.8733 39.37 0)
+			(effects
+				(font
+					(size 1.27 1.27)
+				)
+				(justify left)
+			)
+		)
+		(property "Value" "ESP32-S3-WROOM-1"
+			(at 127.8733 41.91 0)
+			(effects
+				(font
+					(size 1.27 1.27)
+				)
+				(justify left)
+			)
+		)
+		(property "Footprint" "RF_Module:ESP32-S3-WROOM-1"
+			(at 125.73 67.31 0)
+			(effects
+				(font
+					(size 1.27 1.27)
+				)
+				(hide yes)
+			)
+		)
+		(property "Datasheet" "https://www.espressif.com/sites/default/files/documentation/esp32-s3-wroom-1_wroom-1u_datasheet_en.pdf"
+			(at 125.73 69.85 0)
+			(effects
+				(font
+					(size 1.27 1.27)
+				)
+				(hide yes)
+			)
+		)
+		(property "Description" "RF Module, ESP32-S3 SoC, Wi-Fi 802.11b/g/n, Bluetooth, BLE, 32-bit, 3.3V, onboard antenna, SMD"
+			(at 125.73 69.85 0)
+			(effects
+				(font
+					(size 1.27 1.27)
+				)
+				(hide yes)
+			)
+		)
+		(pin "3"
+		)
+		(pin "4"
+		)
+		(pin "15"
+		)
+		(pin "27"
+		)
+		(pin "38"
+		)
+		(pin "39"
+		)
+		(pin "6"
+		)
+		(pin "5"
+		)
+		(pin "7"
+		)
+		(pin "12"
+		)
+		(pin "17"
+		)
+		(pin "19"
+		)
+		(pin "14"
+		)
+		(pin "20"
+		)
+		(pin "23"
+		)
+		(pin "10"
+		)
+		(pin "9"
+		)
+		(pin "16"
+		)
+		(pin "30"
+		)
+		(pin "22"
+		)
+		(pin "8"
+		)
+		(pin "21"
+		)
+		(pin "1"
+		)
+		(pin "36"
+		)
+		(pin "40"
+		)
+		(pin "18"
+		)
+		(pin "2"
+		)
+		(pin "32"
+		)
+		(pin "37"
+		)
+		(pin "11"
+		)
+		(pin "13"
+		)
+		(pin "31"
+		)
+		(pin "29"
+		)
+		(pin "41"
+		)
+		(pin "33"
+		)
+		(pin "34"
+		)
+		(pin "35"
+		)
+		(pin "28"
+		)
+		(pin "26"
+		)
+		(pin "24"
+		)
+		(pin "25"
+		)
+		(instances
+			(project ""
+				(path "/903e2e1f-69db-4eea-89f5-cdb0bf721490"
+					(reference "U1")
+					(unit 1)
+				)
+			)
+		)
+	)
 	(sheet_instances
 		(path "/"
