File: hardware/kicad/heatsinklab.kicad_pcb (KiCad board)
At the start: 2 copper layers, 160 x 120 mm, 20 parts, among them J1 PWR_IN 12V, J10 EXT1 Future, J2 HEATER_OUT, J4 FAN_OUT, J5 FAN_PWM GPIO5, J6 THERMO MAX6675, J7 INA226 0x41, J8 SDP510 0x40, J9 EZO-HUM 0x6F, Q1 IRLZ44N Heater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

Commit message: Update PCB: proper ESP32-S3-DevKitC-1 2x22 pin footprint with correct GPIO net assignments
Replace old 13-pin placeholder with two 22-pin headers matching the
DevKitC-1 pinout. Left header: 3V3(L1-2), GPIO4(L4), GPIO5(L5),
GPIO15/SDA(L8), GPIO16/SCL(L9), GPIO10(L16), GPIO11/MISO(L17),
GPIO12/CS(L18), GPIO13/SCK(L19), GND(L22). Right header: GND(R1,R21-22).
Row spacing 22.86mm matching physical board.

https://claude.ai/code/session_01WnNzHJgAA7wxew4mtPpYTu
Parts:
- added U1-R: ESP32-S3-DevKitC-1 Right, Connector_PinHeader_2.54mm:PinHeader_1x22_P2.54mm_Vertical, F.Cu at (94.9, 23.0)
- U1-L: value ESP32-S3 Left Header -> ESP32-S3-DevKitC-1 Left; footprint Connector_PinHeader_2.54mm:PinHeader_1x13_P2.54mm_Vertical -> Connector_PinHeader_2.54mm:PinHeader_1x22_P2.54mm_Vertical
- moved U1-L 37.9 mm to (72.0, 23.0)
Connections:
- U1-L pad 1: (no net) -> +3.3V
- U1-L pad 10: SPI_CS -> (no net)
- U1-L pad 11: SPI_SCK -> (no net)
- U1-L pad 12: I2C_SDA -> (no net)
- U1-L pad 13: I2C_SCL -> (no net)
- U1-L pad 2: (no net) -> +3.3V
- U1-L pad 4: +3.3V -> GPIO4_HEAT
- U1-L pad 5: GND -> GPIO5_FPWM
- U1-L pad 6: GPIO4_HEAT -> (no net)
- U1-L pad 7: GPIO5_FPWM -> (no net)
- U1-L pad 8: GPIO10_FEN -> I2C_SDA
- U1-L pad 9: SPI_MISO -> I2C_SCL
Changed lines of the file:
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@@
     (pad "2" thru_hole circle (at  5.08 0) (size 1.8 1.8) (drill 0.8) (layers "*.Cu" "*.Mask") (net 2 "GND"))
   )
-  (footprint "Connector_PinHeader_2.54mm:PinHeader_1x13_P2.54mm_Vertical" (layer "F.Cu") (at 80 60) (uuid "fp-esp-left")
-    (property "Reference" "U1-L" (at -5 0 90) (layer "F.SilkS") (effects (font (size 1 1))))
-    (property "Value" "ESP32-S3 Left Header" (at 5 0 90) (layer "F.Fab") (effects (font (size 1 1))))
-    (pad "1"  thru_hole circle (at 0  0   ) (size 1.8 1.8) (drill 1.0) (layers "*.Cu" "*.Mask") (net 0 ""))
-    (pad "2"  thru_hole circle (at 0  2.54) (size 1.8 1.8) (drill 1.0) (layers "*.Cu" "*.Mask") (net 0 ""))
-    (pad "3"  thru_hole circle (at 0  5.08) (size 1.8 1.8) (drill 1.0) (layers "*.Cu" "*.Mask") (net 0 ""))
-    (pad "4"  thru_hole circle (at 0  7.62) (size 1.8 1.8) (drill 1.0) (layers "*.Cu" "*.Mask") (net 13 "+3.3V"))
-    (pad "5"  thru_hole circle (at 0 10.16) (size 1.8 1.8) (drill 1.0) (layers "*.Cu" "*.Mask") (net 2 "GND"))
-    (pad "6"  thru_hole circle (at 0 12.70) (size 1.8 1.8) (drill 1.0) (layers "*.Cu" "*.Mask") (net 5 "GPIO4_HEAT"))
-    (pad "7"  thru_hole circle (at 0 15.24) (size 1.8 1.8) (drill 1.0) (layers "*.Cu" "*.Mask") (net 6 "GPIO5_FPWM"))
-    (pad "8"  thru_hole circle (at 0 17.78) (size 1.8 1.8) (drill 1.0) (layers "*.Cu" "*.Mask") (net 7 "GPIO10_FEN"))
-    (pad "9"  thru_hole circle (at 0 20.32) (size 1.8 1.8) (drill 1.0) (layers "*.Cu" "*.Mask") (net 8 "SPI_MISO"))
-    (pad "10" thru_hole circle (at 0 22.86) (size 1.8 1.8) (drill 1.0) (layers "*.Cu" "*.Mask") (net 9 "SPI_CS"))
-    (pad "11" thru_hole circle (at 0 25.40) (size 1.8 1.8) (drill 1.0) (layers "*.Cu" "*.Mask") (net 10 "SPI_SCK"))
-    (pad "12" thru_hole circle (at 0 27.94) (size 1.8 1.8) (drill 1.0) (layers "*.Cu" "*.Mask") (net 11 "I2C_SDA"))
-    (pad "13" thru_hole circle (at 0 30.48) (size 1.8 1.8) (drill 1.0) (layers "*.Cu" "*.Mask") (net 12 "I2C_SCL"))
+  (footprint "Connector_PinHeader_2.54mm:PinHeader_1x22_P2.54mm_Vertical" (layer "F.Cu") (at 72 23) (uuid "fp-esp-left")
+    (property "Reference" "U1-L" (at -4 26.67 90) (layer "F.SilkS") (effects (font (size 1 1))))
+    (property "Value" "ESP32-S3-DevKitC-1 Left" (at 4 26.67 90) (layer "F.Fab") (effects (font (size 1 1))))
+    (pad "1"  thru_hole rect   (at 0  0    ) (size 1.8 1.8) (drill 1.0) (layers "*.Cu" "*.Mask") (net 13 "+3.3V"))
+    (pad "2"  thru_hole circle (at 0  2.54 ) (size 1.8 1.8) (drill 1.0) (layers "*.Cu" "*.Mask") (net 13 "+3.3V"))
+    (pad "3"  thru_hole circle (at 0  5.08 ) (size 1.8 1.8) (drill 1.0) (layers "*.Cu" "*.Mask") (net 0 ""))
+    (pad "4"  thru_hole circle (at 0  7.62 ) (size 1.8 1.8) (drill 1.0) (layers "*.Cu" "*.Mask") (net 5 "GPIO4_HEAT"))
+    (pad "5"  thru_hole circle (at 0 10.16 ) (size 1.8 1.8) (drill 1.0) (layers "*.Cu" "*.Mask") (net 6 "GPIO5_FPWM"))
+    (pad "6"  thru_hole circle (at 0 12.70 ) (size 1.8 1.8) (drill 1.0) (layers "*.Cu" "*.Mask") (net 0 ""))
+    (pad "7"  thru_hole circle (at 0 15.24 ) (size 1.8 1.8) (drill 1.0) (layers "*.Cu" "*.Mask") (net 0 ""))
+    (pad "8"  thru_hole circle (at 0 17.78 ) (size 1.8 1.8) (drill 1.0) (layers "*.Cu" "*.Mask") (net 11 "I2C_SDA"))
+    (pad "9"  thru_hole circle (at 0 20.32 ) (size 1.8 1.8) (drill 1.0) (layers "*.Cu" "*.Mask") (net 12 "I2C_SCL"))
+    (pad "10" thru_hole circle (at 0 22.86 ) (size 1.8 1.8) (drill 1.0) (layers "*.Cu" "*.Mask") (net 0 ""))
+    (pad "11" thru_hole circle (at 0 25.40 ) (size 1.8 1.8) (drill 1.0) (layers "*.Cu" "*.Mask") (net 0 ""))
+    (pad "12" thru_hole circle (at 0 27.94 ) (size 1.8 1.8) (drill 1.0) (layers "*.Cu" "*.Mask") (net 0 ""))
+    (pad "13" thru_hole circle (at 0 30.48 ) (size 1.8 1.8) (drill 1.0) (layers "*.Cu" "*.Mask") (net 0 ""))
+    (pad "14" thru_hole circle (at 0 33.02 ) (size 1.8 1.8) (drill 1.0) (layers "*.Cu" "*.Mask") (net 0 ""))
+    (pad "15" thru_hole circle (at 0 35.56 ) (size 1.8 1.8) (drill 1.0) (layers "*.Cu" "*.Mask") (net 0 ""))
+    (pad "16" thru_hole circle (at 0 38.10 ) (size 1.8 1.8) (drill 1.0) (layers "*.Cu" "*.Mask") (net 7 "GPIO10_FEN"))
+    (pad "17" thru_hole circle (at 0 40.64 ) (size 1.8 1.8) (drill 1.0) (layers "*.Cu" "*.Mask") (net 8 "SPI_MISO"))
+    (pad "18" thru_hole circle (at 0 43.18 ) (size 1.8 1.8) (drill 1.0) (layers "*.Cu" "*.Mask") (net 9 "SPI_CS"))
+    (pad "19" thru_hole circle (at 0 45.72 ) (size 1.8 1.8) (drill 1.0) (layers "*.Cu" "*.Mask") (net 10 "SPI_SCK"))
+    (pad "20" thru_hole circle (at 0 48.26 ) (size 1.8 1.8) (drill 1.0) (layers "*.Cu" "*.Mask") (net 0 ""))
+    (pad "21" thru_hole circle (at 0 50.80 ) (size 1.8 1.8) (drill 1.0) (layers "*.Cu" "*.Mask") (net 0 ""))
+    (pad "22" thru_hole circle (at 0 53.34 ) (size 1.8 1.8) (drill 1.0) (layers "*.Cu" "*.Mask") (net 2 "GND"))
+  )
+  (footprint "Connector_PinHeader_2.54mm:PinHeader_1x22_P2.54mm_Vertical" (layer "F.Cu") (at 94.86 23) (uuid "fp-esp-right")
+    (property "Reference" "U1-R" (at -4 26.67 90) (layer "F.SilkS") (effects (font (size 1 1))))
+    (property "Value" "ESP32-S3-DevKitC-1 Right" (at 4 26.67 90) (layer "F.Fab") (effects (font (size 1 1))))
+    (pad "1"  thru_hole rect   (at 0  0    ) (size 1.8 1.8) (drill 1.0) (layers "*.Cu" "*.Mask") (net 2 "GND"))
+    (pad "2"  thru_hole circle (at 0  2.54 ) (size 1.8 1.8) (drill 1.0) (layers "*.Cu" "*.Mask") (net 0 ""))
+    (pad "3"  thru_hole circle (at 0  5.08 ) (size 1.8 1.8) (drill 1.0) (layers "*.Cu" "*.Mask") (net 0 ""))
+    (pad "4"  thru_hole circle (at 0  7.62 ) (size 1.8 1.8) (drill 1.0) (layers "*.Cu" "*.Mask") (net 0 ""))
+    (pad "5"  thru_hole circle (at 0 10.16 ) (size 1.8 1.8) (drill 1.0) (layers "*.Cu" "*.Mask") (net 0 ""))
+    (pad "6"  thru_hole circle (at 0 12.70 ) (size 1.8 1.8) (drill 1.0) (layers "*.Cu" "*.Mask") (net 0 ""))
+    (pad "7"  thru_hole circle (at 0 15.24 ) (size 1.8 1.8) (drill 1.0) (layers "*.Cu" "*.Mask") (net 0 ""))
+    (pad "8"  thru_hole circle (at 0 17.78 ) (size 1.8 1.8) (drill 1.0) (layers "*.Cu" "*.Mask") (net 0 ""))
+    (pad "9"  thru_hole circle (at 0 20.32 ) (size 1.8 1.8) (drill 1.0) (layers "*.Cu" "*.Mask") (net 0 ""))
+    (pad "10" thru_hole circle (at 0 22.86 ) (size 1.8 1.8) (drill 1.0) (layers "*.Cu" "*.Mask") (net 0 ""))
+    (pad "11" thru_hole circle (at 0 25.40 ) (size 1.8 1.8) (drill 1.0) (layers "*.Cu" "*.Mask") (net 0 ""))
+    (pad "12" thru_hole circle (at 0 27.94 ) (size 1.8 1.8) (drill 1.0) (layers "*.Cu" "*.Mask") (net 0 ""))
+    (pad "13" thru_hole circle (at 0 30.48 ) (size 1.8 1.8) (drill 1.0) (layers "*.Cu" "*.Mask") (net 0 ""))
+    (pad "14" thru_hole circle (at 0 33.02 ) (size 1.8 1.8) (drill 1.0) (layers "*.Cu" "*.Mask") (net 0 ""))
+    (pad "15" thru_hole circle (at 0 35.56 ) (size 1.8 1.8) (drill 1.0) (layers "*.Cu" "*.Mask") (net 0 ""))
+    (pad "16" thru_hole circle (at 0 38.10 ) (size 1.8 1.8) (drill 1.0) (layers "*.Cu" "*.Mask") (net 0 ""))
+    (pad "17" thru_hole circle (at 0 40.64 ) (size 1.8 1.8) (drill 1.0) (layers "*.Cu" "*.Mask") (net 0 ""))
+    (pad "18" thru_hole circle (at 0 43.18 ) (size 1.8 1.8) (drill 1.0) (layers "*.Cu" "*.Mask") (net 0 ""))
+    (pad "19" thru_hole circle (at 0 45.72 ) (size 1.8 1.8) (drill 1.0) (layers "*.Cu" "*.Mask") (net 0 ""))
+    (pad "20" thru_hole circle (at 0 48.26 ) (size 1.8 1.8) (drill 1.0) (layers "*.Cu" "*.Mask") (net 0 ""))
+    (pad "21" thru_hole circle (at 0 50.80 ) (size 1.8 1.8) (drill 1.0) (layers "*.Cu" "*.Mask") (net 2 "GND"))
+    (pad "22" thru_hole circle (at 0 53.34 ) (size 1.8 1.8) (drill 1.0) (layers "*.Cu" "*.Mask") (net 2 "GND"))
   )
   (gr_text "HeatsinkLab Wind Tunnel" (at 80 5) (layer "F.SilkS") (uuid "title-text")

Commit message: Merge FAN_OUT + FAN_PWM into single 3-pin JST-XH connector J4
J4 now carries: pin1=12V(via Q2), pin2=GND, pin3=GPIO5_PWM.
Removes separate J5 2-pin connector. Adds Conn_01x03 lib symbol.
Updates PCB footprint to JST_XH_B3B-XH-A and wiring schematic doc.

https://claude.ai/code/session_01WnNzHJgAA7wxew4mtPpYTu
Parts:
- removed J5: FAN_PWM GPIO5, Connector_JST:JST_XH_B2B-XH-A_1x02_P2.50mm_Vertical
- J4: value FAN_OUT -> FAN 12V/GND/PWM; footprint Connector_JST:JST_XH_B2B-XH-A_1x02_P2.50mm_Vertical -> Connector_JST:JST_XH_B3B-XH-A_1x03_P2.50mm_Vertical
- moved J4 2.00 mm to (12.0, 52.0)
Changed lines of the file:
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@@
     (pad "2" thru_hole circle (at  1.25 0) (size 2.5 2.5) (drill 1.0) (layers "*.Cu" "*.Mask") (net 2 "GND"))
   )
-  (footprint "Connector_JST:JST_XH_B2B-XH-A_1x02_P2.50mm_Vertical" (layer "F.Cu") (at 12 50) (uuid "fp-j4")
+  (footprint "Connector_JST:JST_XH_B3B-XH-A_1x03_P2.50mm_Vertical" (layer "F.Cu") (at 12 52) (uuid "fp-j4")
     (property "Reference" "J4" (at 0 -4 0) (layer "F.SilkS") (effects (font (size 1 1))))
-    (property "Value" "FAN_OUT" (at 0 4.5 0) (layer "F.Fab") (effects (font (size 1 1))))
-    (pad "1" thru_hole rect   (at -1.25 0) (size 2.5 2.5) (drill 1.0) (layers "*.Cu" "*.Mask") (net 4 "FAN_OUT_P"))
-    (pad "2" thru_hole circle (at  1.25 0) (size 2.5 2.5) (drill 1.0) (layers "*.Cu" "*.Mask") (net 2 "GND"))
-  )
-  (footprint "Connector_JST:JST_XH_B2B-XH-A_1x02_P2.50mm_Vertical" (layer "F.Cu") (at 12 65) (uuid "fp-j5")
-    (property "Reference" "J5" (at 0 -4 0) (layer "F.SilkS") (effects (font (size 1 1))))
-    (property "Value" "FAN_PWM GPIO5" (at 0 4.5 0) (layer "F.Fab") (effects (font (size 1 1))))
-    (pad "1" thru_hole rect   (at -1.25 0) (size 2.5 2.5) (drill 1.0) (layers "*.Cu" "*.Mask") (net 6 "GPIO5_FPWM"))
-    (pad "2" thru_hole circle (at  1.25 0) (size 2.5 2.5) (drill 1.0) (layers "*.Cu" "*.Mask") (net 2 "GND"))
+    (property "Value" "FAN 12V/GND/PWM" (at 0 5 0) (layer "F.Fab") (effects (font (size 1 1))))
+    (pad "1" thru_hole rect   (at -2.5 0) (size 2.5 2.5) (drill 1.0) (layers "*.Cu" "*.Mask") (net 4 "FAN_OUT_P"))
+    (pad "2" thru_hole circle (at  0   0) (size 2.5 2.5) (drill 1.0) (layers "*.Cu" "*.Mask") (net 2 "GND"))
+    (pad "3" thru_hole circle (at  2.5 0) (size 2.5 2.5) (drill 1.0) (layers "*.Cu" "*.Mask") (net 6 "GPIO5_FPWM"))
   )
   (footprint "Connector_JST:JST_XH_B5B-XH-A_1x05_P2.50mm_Vertical" (layer "F.Cu") (at 148 15) (uuid "fp-j6")
